File: kicad/ECE533_Guide/controller.kicad_sch (KiCad schematic)
At the start: 39 parts, among them U16 SN74LVC1G74, U17 SN74LVC1G74, U19 74LVC1G08, U20 74LVC1G08, U5 LTC3861IUHE#PBF

Commit message: Stage 2: BOM from schematic, LCSC numbers, fix duplicate C114 (refs #2)
- kicad/tools/make_bom.py builds bom/PCB_BOM.xlsx (+ CSV) from the netlist;
  previous report BOM kept as a sheet, Digi-Key PNs carried over
- 47 LCSC numbers verified on lcsc.com; two unconfirmed Murata MPNs replaced
- check_netlist.py now also checks for duplicate reference designators
- Yageo part-number codes fixed (13K, 0R jumper)

Co-Authored-By: Claude Opus 5.5 <noreply@anthropic.com>
Parts:
- C101: LCSC (none) -> C86020
- C102, C103, C111, C112, C113, C114: LCSC (none) -> C77055
- C104, C109: LCSC (none) -> C71664
- C105, C106: LCSC (none) -> C77026
- C107: LCSC (none) -> C86023
- C108: LCSC (none) -> C77057
Changed lines of the file:
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@@
 		(property "MPN" "GRM188R71E105KA12D" (at 177.8 80.01 0) (hide yes) (effects (font (size 1.27 1.27))))
 		(property "Manufacturer" "Murata" (at 177.8 80.01 0) (hide yes) (effects (font (size 1.27 1.27))))
+		(property "LCSC" "C86020" (at 177.8 80.01 0) (hide yes) (effects (font (size 1.27 1.27))))
 		(pin "1")
 		(pin "2")
@@
 		(property "MPN" "GRM188R71H104KA93D" (at 187.96 80.01 0) (hide yes) (effects (font (size 1.27 1.27))))
 		(property "Manufacturer" "Murata" (at 187.96 80.01 0) (hide yes) (effects (font (size 1.27 1.27))))
+		(property "LCSC" "C77055" (at 187.96 80.01 0) (hide yes) (effects (font (size 1.27 1.27))))
 		(pin "1")
 		(pin "2")
@@
 		(property "MPN" "GRM188R71H104KA93D" (at 43.18 49.53 0) (hide yes) (effects (font (size 1.27 1.27))))
 		(property "Manufacturer" "Murata" (at 43.18 49.53 0) (hide yes) (effects (font (size 1.27 1.27))))
+		(property "LCSC" "C77055" (at 43.18 49.53 0) (hide yes) (effects (font (size 1.27 1.27))))
 		(pin "1")
 		(pin "2")
@@
 		(property "MPN" "GRM1885C1H101JA01D" (at 81.28 49.53 0) (hide yes) (effects (font (size 1.27 1.27))))
 		(property "Manufacturer" "Murata" (at 81.28 49.53 0) (hide yes) (effects (font (size 1.27 1.27))))
+		(property "LCSC" "C71664" (at 81.28 49.53 0) (hide yes) (effects (font (size 1.27 1.27))))
 		(pin "1")
 		(pin "2")
@@
 		(property "MPN" "GRM1885C1H102JA01D" (at 86.36 171.45 0) (hide yes) (effects (font (size 1.27 1.27))))
 		(property "Manufacturer" "Murata" (at 86.36 171.45 0) (hide yes) (effects (font (size 1.27 1.27))))
+		(property "LCSC" "C77026" (at 86.36 171.45 0) (hide yes) (effects (font (size 1.27 1.27))))
 		(pin "1")
 		(pin "2")
@@
 		(property "MPN" "GRM1885C1H102JA01D" (at 86.36 222.25 0) (hide yes) (effects (font (size 1.27 1.27))))
 		(property "Manufacturer" "Murata" (at 86.36 222.25 0) (hide yes) (effects (font (size 1.27 1.27))))
+		(property "LCSC" "C77026" (at 86.36 222.25 0) (hide yes) (effects (font (size 1.27 1.27))))
 		(pin "1")
 		(pin "2")
@@
 		(property "MPN" "GRM188R71H222KA01D" (at 242.57 127 90) (hide yes) (effects (font (size 1.27 1.27))))
 		(property "Manufacturer" "Murata" (at 242.57 127 90) (hide yes) (effects (font (size 1.27 1.27))))
+		(property "LCSC" "C86023" (at 242.57 127 90) (hide yes) (effects (font (size 1.27 1.27))))
 		(pin "1")
 		(pin "2")
@@
 		(property "MPN" "GRM188R71H472KA01D" (at 242.57 142.24 90) (hide yes) (effects (font (size 1.27 1.27))))
 		(property "Manufacturer" "Murata" (at 242.57 142.24 90) (hide yes) (effects (font (size 1.27 1.27))))
+		(property "LCSC" "C77057" (at 242.57 142.24 90) (hide yes) (effects (font (size 1.27 1.27))))
 		(pin "1")
 		(pin "2")
@@
 		(property "MPN" "GRM1885C1H101JA01D" (at 231.14 152.4 90) (hide yes) (effects (font (size 1.27 1.27))))
 		(property "Manufacturer" "Murata" (at 231.14 152.4 90) (hide yes) (effects (font (size 1.27 1.27))))
+		(property "LCSC" "C71664" (at 231.14 152.4 90) (hide yes) (effects (font (size 1.27 1.27))))
 		(pin "1")
 		(pin "2")
@@
 		(property "MPN" "GRM188R71H104KA93D" (at 289.56 54.61 0) (hide yes) (effects (font (size 1.27 1.27))))
 		(property "Manufacturer" "Murata" (at 289.56 54.61 0) (hide yes) (effects (font (size 1.27 1.27))))
+		(property "LCSC" "C77055" (at 289.56 54.61 0) (hide yes) (effects (font (size 1.27 1.27))))
 		(pin "1")
 		(pin "2")
@@
 		(property "MPN" "GRM188R71H104KA93D" (at 350.52 54.61 0) (hide yes) (effects (font (size 1.27 1.27))))
 		(property "Manufacturer" "Murata" (at 350.52 54.61 0) (hide yes) (effects (font (size 1.27 1.27))))
+		(property "LCSC" "C77055" (at 350.52 54.61 0) (hide yes) (effects (font (size 1.27 1.27))))
 		(pin "1")
 		(pin "2")
@@
 		(property "MPN" "GRM188R71H104KA93D" (at 289.56 115.57 0) (hide yes) (effects (font (size 1.27 1.27))))
 		(property "Manufacturer" "Murata" (at 289.56 115.57 0) (hide yes) (effects (font (size 1.27 1.27))))
+		(property "LCSC" "C77055" (at 289.56 115.57 0) (hide yes) (effects (font (size 1.27 1.27))))
 		(pin "1")
 		(pin "2")
@@
 		(property "MPN" "GRM188R71H104KA93D" (at 350.52 115.57 0) (hide yes) (effects (font (size 1.27 1.27))))
 		(property "Manufacturer" "Murata" (at 350.52 115.57 0) (hide yes) (effects (font (size 1.27 1.27))))
-		(pin "1")
-		(pin "2")
+		(property "LCSC" "C77055" (at 350.52 115.57 0) (hide yes) (effects (font (size 1.27 1.27))))
+		(pin "1")
+		(pin "2")
