File: kicad/ECE533_Guide/fault_io.kicad_sch (KiCad schematic)
At the start: 24 parts, among them J4 RACK I/O Nano-Fit, Q7 2N7002, Q8 2N7002, U15 TLV3012, U18 SN74LVC1G74, U25 74LVC1G08

Commit message: Stage 2: BOM from schematic, LCSC numbers, fix duplicate C114 (refs #2)
- kicad/tools/make_bom.py builds bom/PCB_BOM.xlsx (+ CSV) from the netlist;
  previous report BOM kept as a sheet, Digi-Key PNs carried over
- 47 LCSC numbers verified on lcsc.com; two unconfirmed Murata MPNs replaced
- check_netlist.py now also checks for duplicate reference designators
- Yageo part-number codes fixed (13K, 0R jumper)

Co-Authored-By: Claude Opus 5.5 <noreply@anthropic.com>
Parts:
- removed C114: 100n/50V, Capacitor_SMD:C_0603_1608Metric, symbol Device:C
- added C119: 100n/50V, Capacitor_SMD:C_0603_1608Metric, symbol Device:C
- C115: LCSC (none) -> C86020
- C116, C117: LCSC (none) -> C77055
- C118: LCSC (none) -> C77053
- D15, D16: LCSC (none) -> C134417
- D8: LCSC (none) -> C125098
- D9: LCSC (none) -> C125099
- Q7, Q8: LCSC (none) -> C16338
Connections:
- net +5V_ISO: now also C119.1
- net GND_ISO: now also C119.2
Changed lines of the file:
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@@
 		(on_board yes)
 		(dnp no)
-		(property "Reference" "C114" (at 114.3 48.26 0) (effects (font (size 1.27 1.27)) (justify left)))
+		(property "Reference" "C119" (at 114.3 48.26 0) (effects (font (size 1.27 1.27)) (justify left)))
 		(property "Value" "100n/50V" (at 114.3 50.8 0) (effects (font (size 1.27 1.27)) (justify left)))
 		(property "Footprint" "Capacitor_SMD:C_0603_1608Metric" (at 111.76 49.53 0) (hide yes) (effects (font (size 1.27 1.27))))
@@
 		(property "MPN" "GRM188R71H104KA93D" (at 111.76 49.53 0) (hide yes) (effects (font (size 1.27 1.27))))
 		(property "Manufacturer" "Murata" (at 111.76 49.53 0) (hide yes) (effects (font (size 1.27 1.27))))
-		(pin "1")
-		(pin "2")
-		(instances (project "ECE533_Guide"
-			(path "/3bc94f09-386f-53fd-bc70-05d96028f503/d6cd4086-c11b-5611-86b3-40ade4c6962b/fc36bed8-9c54-58f8-b7ac-38dffeea96ea" (reference "C114") (unit 1))
+		(property "LCSC" "C77055" (at 111.76 49.53 0) (hide yes) (effects (font (size 1.27 1.27))))
+		(pin "1")
+		(pin "2")
+		(instances (project "ECE533_Guide"
+			(path "/3bc94f09-386f-53fd-bc70-05d96028f503/d6cd4086-c11b-5611-86b3-40ade4c6962b/fc36bed8-9c54-58f8-b7ac-38dffeea96ea" (reference "C119") (unit 1))
 		))
 	)
@@
 		(property "MPN" "GRM188R71E105KA12D" (at 193.04 102.87 0) (hide yes) (effects (font (size 1.27 1.27))))
 		(property "Manufacturer" "Murata" (at 193.04 102.87 0) (hide yes) (effects (font (size 1.27 1.27))))
+		(property "LCSC" "C86020" (at 193.04 102.87 0) (hide yes) (effects (font (size 1.27 1.27))))
 		(pin "1")
 		(pin "2")
@@
 		(property "MPN" "GRM188R71H104KA93D" (at 254 49.53 0) (hide yes) (effects (font (size 1.27 1.27))))
 		(property "Manufacturer" "Murata" (at 254 49.53 0) (hide yes) (effects (font (size 1.27 1.27))))
+		(property "LCSC" "C77055" (at 254 49.53 0) (hide yes) (effects (font (size 1.27 1.27))))
 		(pin "1")
 		(pin "2")
@@
 		(property "MPN" "GRM188R71H104KA93D" (at 182.88 49.53 0) (hide yes) (effects (font (size 1.27 1.27))))
 		(property "Manufacturer" "Murata" (at 182.88 49.53 0) (hide yes) (effects (font (size 1.27 1.27))))
+		(property "LCSC" "C77055" (at 182.88 49.53 0) (hide yes) (effects (font (size 1.27 1.27))))
 		(pin "1")
 		(pin "2")
@@
 		(property "MPN" "GRM188R71H103KA01D" (at 325.12 64.77 0) (hide yes) (effects (font (size 1.27 1.27))))
 		(property "Manufacturer" "Murata" (at 325.12 64.77 0) (hide yes) (effects (font (size 1.27 1.27))))
+		(property "LCSC" "C77053" (at 325.12 64.77 0) (hide yes) (effects (font (size 1.27 1.27))))
 		(pin "1")
 		(pin "2")
@@
 		(property "MPN" "BAT54W-7-F" (at 320.04 81.28 0) (hide yes) (effects (font (size 1.27 1.27))))
 		(property "Manufacturer" "Diodes Inc" (at 320.04 81.28 0) (hide yes) (effects (font (size 1.27 1.27))))
+		(property "LCSC" "C134417" (at 320.04 81.28 0) (hide yes) (effects (font (size 1.27 1.27))))
 		(pin "1")
 		(pin "2")
@@
 		(property "MPN" "BAT54W-7-F" (at 320.04 93.98 0) (hide yes) (effects (font (size 1.27 1.27))))
 		(property "Manufacturer" "Diodes Inc" (at 320.04 93.98 0) (hide yes) (effects (font (size 1.27 1.27))))
+		(property "LCSC" "C134417" (at 320.04 93.98 0) (hide yes) (effects (font (size 1.27 1.27))))
 		(pin "1")
 		(pin "2")
@@
 		(property "MPN" "LTST-C191KRKT" (at 41.91 172.72 0) (hide yes) (effects (font (size 1.27 1.27))))
 		(property "Manufacturer" "Lite-On" (at 41.91 172.72 0) (hide yes) (effects (font (size 1.27 1.27))))
+		(property "LCSC" "C125099" (at 41.91 172.72 0) (hide yes) (effects (font (size 1.27 1.27))))
 		(pin "1")
 		(pin "2")
@@
 		(property "MPN" "LTST-C191KGKT" (at 41.91 198.12 0) (hide yes) (effects (font (size 1.27 1.27))))
 		(property "Manufacturer" "Lite-On" (at 41.91 198.12 0) (hide yes) (effects (font (size 1.27 1.27))))
+		(property "LCSC" "C125098" (at 41.91 198.12 0) (hide yes) (effects (font (size 1.27 1.27))))
 		(pin "1")
 		(pin "2")
@@
 		(property "MPN" "2N7002LT1G" (at 101.6 218.44 0) (hide yes) (effects (font (size 1.27 1.27))))
 		(property "Manufacturer" "onsemi" (at 101.6 218.44 0) (hide yes) (effects (font (size 1.27 1.27))))
+		(property "LCSC" "C16338" (at 101.6 218.44 0) (hide yes) (effects (font (size 1.27 1.27))))
 		(pin "1")
 		(pin "2")
@@
 		(property "MPN" "2N7002LT1G" (at 162.56 218.44 0) (hide yes) (effects (font (size 1.27 1.27))))
 		(property "Manufacturer" "onsemi" (at 162.56 218.44 0) (hide yes) (effects (font (size 1.27 1.27))))
-		(pin "1")
-		(pin "2")
+		(property "LCSC" "C16338" (at 162.56 218.44 0) (hide yes) (effects (font (size 1.27 1.27))))
+		(pin "1")
+		(pin "2")

Commit message: Stage 3: footprints from datasheets and vendor libraries, 3D-checked (refs #3)
- ECE533_Mods.pretty (drawn from manufacturer datasheets):
  EPC2304 (EPC copper, solder-mask-defined land pattern and stencil),
  TDK ERUC23 (TDK recommended layout), R_2512_Kelvin (Bourns CSS2H-2512
  pads with net-tie sense strips), Littelfuse 456 fuse (+ placeholder STEP)
- ECE533_Vendor library (git-ignored): Wurth REDCUBE 74650194R and the
  SamacSys NME1S0505SC footprint; vendor STEP models referenced from
  kicad/lib/vendor, alignment verified by rendering
- gen_footprints.py regenerates both libraries; check_footprints.py checks
  symbol pins against footprint pads
- Fix D15/D16 BAT54W footprint: SOT-323, not SOD-323 (pin 3 had no pad)
- ERC: 0 violations locally (footprint links now resolve)

Co-Authored-By: Claude Opus 5.5 <noreply@anthropic.com>
Parts:
- D15, D16: footprint Diode_SMD:D_SOD-323 -> Package_TO_SOT_SMD:SOT-323_SC-70
Changed lines of the file:
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@@
 		(property "Reference" "D15" (at 317.5 78.74 0) (effects (font (size 1.27 1.27)) (justify left)))
 		(property "Value" "BAT54W" (at 317.5 85.09 0) (effects (font (size 1.27 1.27)) (justify left)))
-		(property "Footprint" "Diode_SMD:D_SOD-323" (at 320.04 81.28 0) (hide yes) (effects (font (size 1.27 1.27))))
+		(property "Footprint" "Package_TO_SOT_SMD:SOT-323_SC-70" (at 320.04 81.28 0) (hide yes) (effects (font (size 1.27 1.27))))
 		(property "Datasheet" "https://assets.nexperia.com/documents/data-sheet/BAT54W_SER.pdf" (at 320.04 81.28 0) (hide yes) (effects (font (size 1.27 1.27))))
 		(property "Description" "Schottky barrier diode, SOT-323" (at 320.04 81.28 0) (hide yes) (effects (font (size 1.27 1.27))))
@@
 		(property "Reference" "D16" (at 317.5 91.44 0) (effects (font (size 1.27 1.27)) (justify left)))
 		(property "Value" "BAT54W" (at 317.5 97.79 0) (effects (font (size 1.27 1.27)) (justify left)))
-		(property "Footprint" "Diode_SMD:D_SOD-323" (at 320.04 93.98 0) (hide yes) (effects (font (size 1.27 1.27))))
+		(property "Footprint" "Package_TO_SOT_SMD:SOT-323_SC-70" (at 320.04 93.98 0) (hide yes) (effects (font (size 1.27 1.27))))
 		(property "Datasheet" "https://assets.nexperia.com/documents/data-sheet/BAT54W_SER.pdf" (at 320.04 93.98 0) (hide yes) (effects (font (size 1.27 1.27))))
 		(property "Description" "Schottky barrier diode, SOT-323" (at 320.04 93.98 0) (hide yes) (effects (font (size 1.27 1.27))))
