File: kicad/ECE533_Guide/aux_supply_fan.kicad_sch (KiCad schematic)
At the start: 31 parts, among them J5 FAN Micro-Fit, U11 LM5012DDAR, U21 TPS2553DBVR

Commit message: Stage 2: BOM from schematic, LCSC numbers, fix duplicate C114 (refs #2)
- kicad/tools/make_bom.py builds bom/PCB_BOM.xlsx (+ CSV) from the netlist;
  previous report BOM kept as a sheet, Digi-Key PNs carried over
- 47 LCSC numbers verified on lcsc.com; two unconfirmed Murata MPNs replaced
- check_netlist.py now also checks for duplicate reference designators
- Yageo part-number codes fixed (13K, 0R jumper)

Co-Authored-By: Claude Opus 5.5 <noreply@anthropic.com>
Parts:
- C76: LCSC (none) -> C77058
- C77: LCSC (none) -> C86023
- C78, C79: LCSC (none) -> C91604
- C80: LCSC (none) -> C77055
- C81: LCSC (none) -> C77057
- C82: LCSC (none) -> C86027
- C83: LCSC (none) -> C86020
- C84: LCSC (none) -> C86038
Changed lines of the file:
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@@
 		(property "MPN" "GRM188R72A104KA35D" (at 71.12 72.39 0) (hide yes) (effects (font (size 1.27 1.27))))
 		(property "Manufacturer" "Murata" (at 71.12 72.39 0) (hide yes) (effects (font (size 1.27 1.27))))
+		(property "LCSC" "C77058" (at 71.12 72.39 0) (hide yes) (effects (font (size 1.27 1.27))))
 		(pin "1")
 		(pin "2")
@@
 		(property "MPN" "GRM188R71H222KA01D" (at 142.24 49.53 0) (hide yes) (effects (font (size 1.27 1.27))))
 		(property "Manufacturer" "Murata" (at 142.24 49.53 0) (hide yes) (effects (font (size 1.27 1.27))))
+		(property "LCSC" "C86023" (at 142.24 49.53 0) (hide yes) (effects (font (size 1.27 1.27))))
 		(pin "1")
 		(pin "2")
@@
 		(property "MPN" "GRM31CR71A226KE15L" (at 203.2 69.85 0) (hide yes) (effects (font (size 1.27 1.27))))
 		(property "Manufacturer" "Murata" (at 203.2 69.85 0) (hide yes) (effects (font (size 1.27 1.27))))
+		(property "LCSC" "C91604" (at 203.2 69.85 0) (hide yes) (effects (font (size 1.27 1.27))))
 		(pin "1")
 		(pin "2")
@@
 		(property "MPN" "GRM31CR71A226KE15L" (at 213.36 69.85 0) (hide yes) (effects (font (size 1.27 1.27))))
 		(property "Manufacturer" "Murata" (at 213.36 69.85 0) (hide yes) (effects (font (size 1.27 1.27))))
+		(property "LCSC" "C91604" (at 213.36 69.85 0) (hide yes) (effects (font (size 1.27 1.27))))
 		(pin "1")
 		(pin "2")
@@
 		(property "MPN" "GRM188R71H104KA93D" (at 223.52 69.85 0) (hide yes) (effects (font (size 1.27 1.27))))
 		(property "Manufacturer" "Murata" (at 223.52 69.85 0) (hide yes) (effects (font (size 1.27 1.27))))
+		(property "LCSC" "C77055" (at 223.52 69.85 0) (hide yes) (effects (font (size 1.27 1.27))))
 		(pin "1")
 		(pin "2")
@@
 		(property "MPN" "GRM188R71H472KA01D" (at 193.04 100.33 0) (hide yes) (effects (font (size 1.27 1.27))))
 		(property "Manufacturer" "Murata" (at 193.04 100.33 0) (hide yes) (effects (font (size 1.27 1.27))))
+		(property "LCSC" "C77057" (at 193.04 100.33 0) (hide yes) (effects (font (size 1.27 1.27))))
 		(pin "1")
 		(pin "2")
@@
 		(property "MPN" "GRM188R71H473KA61D" (at 213.36 100.33 0) (hide yes) (effects (font (size 1.27 1.27))))
 		(property "Manufacturer" "Murata" (at 213.36 100.33 0) (hide yes) (effects (font (size 1.27 1.27))))
+		(property "LCSC" "C86027" (at 213.36 100.33 0) (hide yes) (effects (font (size 1.27 1.27))))
 		(pin "1")
 		(pin "2")
@@
 		(property "MPN" "GRM188R71E105KA12D" (at 25.4 166.37 0) (hide yes) (effects (font (size 1.27 1.27))))
 		(property "Manufacturer" "Murata" (at 25.4 166.37 0) (hide yes) (effects (font (size 1.27 1.27))))
+		(property "LCSC" "C86020" (at 25.4 166.37 0) (hide yes) (effects (font (size 1.27 1.27))))
 		(pin "1")
 		(pin "2")
@@
 		(property "MPN" "GRM21BR71A106KE51L" (at 132.08 191.77 0) (hide yes) (effects (font (size 1.27 1.27))))
 		(property "Manufacturer" "Murata" (at 132.08 191.77 0) (hide yes) (effects (font (size 1.27 1.27))))
-		(pin "1")
-		(pin "2")
+		(property "LCSC" "C86038" (at 132.08 191.77 0) (hide yes) (effects (font (size 1.27 1.27))))
+		(pin "1")
+		(pin "2")

Commit message: Stage 3: board set-up, JLCPCB rules and first-pass placement (refs #3)
- build_pcb.py builds the PCB from the netlist: ID-1 outline, 4 x 2 oz
  stack-up (3313, ENIG), layer names, LV_ISO/HV_SW net classes, heatsink,
  pedestal and fan-duct outlines, isolation-barrier rule area, and places
  all 273 footprints (power stage on the bottom under L1, isolators on the
  barrier column, terminals on the right edge)
- ECE533_Guide.kicad_dru: JLC 2 oz limits, HV margin, 2.5 mm barrier rule
- Test points 1.0 mm (all on top); L1 pin-1 mark moved off RS2
- DRC with parity: 0 errors; only unrouted nets and 1 silk warning remain
- docs/design/placement_stage3.md with renders, PROGRESS updated

Co-Authored-By: Claude Opus 5.5 <noreply@anthropic.com>
Parts:
- TP12, TP13, TP14: footprint TestPoint:TestPoint_Pad_D1.5mm -> TestPoint:TestPoint_Pad_D1.0mm
Changed lines of the file:
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@@
 		(property "Reference" "TP12" (at 266.7 64.77 0) (effects (font (size 1.27 1.27)) (justify left)))
 		(property "Value" "+5V_PWR" (at 266.7 67.31 0) (effects (font (size 1.27 1.27)) (justify left)))
-		(property "Footprint" "TestPoint:TestPoint_Pad_D1.5mm" (at 264.16 66.04 0) (hide yes) (effects (font (size 1.27 1.27))))
+		(property "Footprint" "TestPoint:TestPoint_Pad_D1.0mm" (at 264.16 66.04 0) (hide yes) (effects (font (size 1.27 1.27))))
 		(property "Datasheet" "" (at 264.16 66.04 0) (hide yes) (effects (font (size 1.27 1.27))))
 		(property "Description" "test point" (at 264.16 66.04 0) (hide yes) (effects (font (size 1.27 1.27))))
@@
 		(property "Reference" "TP13" (at 119.38 171.45 0) (effects (font (size 1.27 1.27)) (justify left)))
 		(property "Value" "FAN_FLT" (at 119.38 173.99 0) (effects (font (size 1.27 1.27)) (justify left)))
-		(property "Footprint" "TestPoint:TestPoint_Pad_D1.5mm" (at 116.84 172.72 0) (hide yes) (effects (font (size 1.27 1.27))))
+		(property "Footprint" "TestPoint:TestPoint_Pad_D1.0mm" (at 116.84 172.72 0) (hide yes) (effects (font (size 1.27 1.27))))
 		(property "Datasheet" "" (at 116.84 172.72 0) (hide yes) (effects (font (size 1.27 1.27))))
 		(property "Description" "test point" (at 116.84 172.72 0) (hide yes) (effects (font (size 1.27 1.27))))
@@
 		(property "Reference" "TP14" (at 175.26 171.45 0) (effects (font (size 1.27 1.27)) (justify left)))
 		(property "Value" "TACH" (at 175.26 173.99 0) (effects (font (size 1.27 1.27)) (justify left)))
-		(property "Footprint" "TestPoint:TestPoint_Pad_D1.5mm" (at 172.72 172.72 0) (hide yes) (effects (font (size 1.27 1.27))))
+		(property "Footprint" "TestPoint:TestPoint_Pad_D1.0mm" (at 172.72 172.72 0) (hide yes) (effects (font (size 1.27 1.27))))
 		(property "Datasheet" "" (at 172.72 172.72 0) (hide yes) (effects (font (size 1.27 1.27))))
 		(property "Description" "test point" (at 172.72 172.72 0) (hide yes) (effects (font (size 1.27 1.27))))
