File: kicad/ECE533_Guide/isolation.kicad_sch (KiCad schematic)
At the start: 24 parts, among them U8 AMC3330

Commit message: Stage 2: BOM from schematic, LCSC numbers, fix duplicate C114 (refs #2)
- kicad/tools/make_bom.py builds bom/PCB_BOM.xlsx (+ CSV) from the netlist;
  previous report BOM kept as a sheet, Digi-Key PNs carried over
- 47 LCSC numbers verified on lcsc.com; two unconfirmed Murata MPNs replaced
- check_netlist.py now also checks for duplicate reference designators
- Yageo part-number codes fixed (13K, 0R jumper)

Co-Authored-By: Claude Opus 5.5 <noreply@anthropic.com>
Parts:
- C100, C87, C88, C89, C90, C91, C94, C96, C98: LCSC (none) -> C77055
- C85, C93, C95, C97, C99: LCSC (none) -> C86020
- C86: LCSC (none) -> C86038
- C92: LCSC (none) -> C71664
Changed lines of the file:
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@@
 		(property "MPN" "GRM188R71E105KA12D" (at 162.56 49.53 0) (hide yes) (effects (font (size 1.27 1.27))))
 		(property "Manufacturer" "Murata" (at 162.56 49.53 0) (hide yes) (effects (font (size 1.27 1.27))))
+		(property "LCSC" "C86020" (at 162.56 49.53 0) (hide yes) (effects (font (size 1.27 1.27))))
 		(pin "1")
 		(pin "2")
@@
 		(property "MPN" "GRM21BR71A106KE51L" (at 238.76 49.53 0) (hide yes) (effects (font (size 1.27 1.27))))
 		(property "Manufacturer" "Murata" (at 238.76 49.53 0) (hide yes) (effects (font (size 1.27 1.27))))
+		(property "LCSC" "C86038" (at 238.76 49.53 0) (hide yes) (effects (font (size 1.27 1.27))))
 		(pin "1")
 		(pin "2")
@@
 		(property "MPN" "GRM188R71H104KA93D" (at 248.92 49.53 0) (hide yes) (effects (font (size 1.27 1.27))))
 		(property "Manufacturer" "Murata" (at 248.92 49.53 0) (hide yes) (effects (font (size 1.27 1.27))))
+		(property "LCSC" "C77055" (at 248.92 49.53 0) (hide yes) (effects (font (size 1.27 1.27))))
 		(pin "1")
 		(pin "2")
@@
 		(property "MPN" "GRM188R71H104KA93D" (at 157.48 97.79 0) (hide yes) (effects (font (size 1.27 1.27))))
 		(property "Manufacturer" "Murata" (at 157.48 97.79 0) (hide yes) (effects (font (size 1.27 1.27))))
+		(property "LCSC" "C77055" (at 157.48 97.79 0) (hide yes) (effects (font (size 1.27 1.27))))
 		(pin "1")
 		(pin "2")
@@
 		(property "MPN" "GRM188R71H104KA93D" (at 248.92 97.79 0) (hide yes) (effects (font (size 1.27 1.27))))
 		(property "Manufacturer" "Murata" (at 248.92 97.79 0) (hide yes) (effects (font (size 1.27 1.27))))
+		(property "LCSC" "C77055" (at 248.92 97.79 0) (hide yes) (effects (font (size 1.27 1.27))))
 		(pin "1")
 		(pin "2")
@@
 		(property "MPN" "GRM188R71H104KA93D" (at 157.48 130.81 0) (hide yes) (effects (font (size 1.27 1.27))))
 		(property "Manufacturer" "Murata" (at 157.48 130.81 0) (hide yes) (effects (font (size 1.27 1.27))))
+		(property "LCSC" "C77055" (at 157.48 130.81 0) (hide yes) (effects (font (size 1.27 1.27))))
 		(pin "1")
 		(pin "2")
@@
 		(property "MPN" "GRM188R71H104KA93D" (at 248.92 130.81 0) (hide yes) (effects (font (size 1.27 1.27))))
 		(property "Manufacturer" "Murata" (at 248.92 130.81 0) (hide yes) (effects (font (size 1.27 1.27))))
+		(property "LCSC" "C77055" (at 248.92 130.81 0) (hide yes) (effects (font (size 1.27 1.27))))
 		(pin "1")
 		(pin "2")
@@
 		(property "MPN" "GRM1885C1H101JA01D" (at 121.92 199.39 0) (hide yes) (effects (font (size 1.27 1.27))))
 		(property "Manufacturer" "Murata" (at 121.92 199.39 0) (hide yes) (effects (font (size 1.27 1.27))))
+		(property "LCSC" "C71664" (at 121.92 199.39 0) (hide yes) (effects (font (size 1.27 1.27))))
 		(pin "1")
 		(pin "2")
@@
 		(property "MPN" "GRM188R71E105KA12D" (at 35.56 181.61 0) (hide yes) (effects (font (size 1.27 1.27))))
 		(property "Manufacturer" "Murata" (at 35.56 181.61 0) (hide yes) (effects (font (size 1.27 1.27))))
+		(property "LCSC" "C86020" (at 35.56 181.61 0) (hide yes) (effects (font (size 1.27 1.27))))
 		(pin "1")
 		(pin "2")
@@
 		(property "MPN" "GRM188R71H104KA93D" (at 48.26 181.61 0) (hide yes) (effects (font (size 1.27 1.27))))
 		(property "Manufacturer" "Murata" (at 48.26 181.61 0) (hide yes) (effects (font (size 1.27 1.27))))
+		(property "LCSC" "C77055" (at 48.26 181.61 0) (hide yes) (effects (font (size 1.27 1.27))))
 		(pin "1")
 		(pin "2")
@@
 		(property "MPN" "GRM188R71E105KA12D" (at 60.96 181.61 0) (hide yes) (effects (font (size 1.27 1.27))))
 		(property "Manufacturer" "Murata" (at 60.96 181.61 0) (hide yes) (effects (font (size 1.27 1.27))))
+		(property "LCSC" "C86020" (at 60.96 181.61 0) (hide yes) (effects (font (size 1.27 1.27))))
 		(pin "1")
 		(pin "2")
@@
 		(property "MPN" "GRM188R71H104KA93D" (at 73.66 181.61 0) (hide yes) (effects (font (size 1.27 1.27))))
 		(property "Manufacturer" "Murata" (at 73.66 181.61 0) (hide yes) (effects (font (size 1.27 1.27))))
+		(property "LCSC" "C77055" (at 73.66 181.61 0) (hide yes) (effects (font (size 1.27 1.27))))
 		(pin "1")
 		(pin "2")
@@
 		(property "MPN" "GRM188R71E105KA12D" (at 248.92 181.61 0) (hide yes) (effects (font (size 1.27 1.27))))
 		(property "Manufacturer" "Murata" (at 248.92 181.61 0) (hide yes) (effects (font (size 1.27 1.27))))
+		(property "LCSC" "C86020" (at 248.92 181.61 0) (hide yes) (effects (font (size 1.27 1.27))))
 		(pin "1")
 		(pin "2")
@@
 		(property "MPN" "GRM188R71H104KA93D" (at 261.62 181.61 0) (hide yes) (effects (font (size 1.27 1.27))))
 		(property "Manufacturer" "Murata" (at 261.62 181.61 0) (hide yes) (effects (font (size 1.27 1.27))))
+		(property "LCSC" "C77055" (at 261.62 181.61 0) (hide yes) (effects (font (size 1.27 1.27))))
 		(pin "1")
 		(pin "2")
@@
 		(property "MPN" "GRM188R71E105KA12D" (at 274.32 181.61 0) (hide yes) (effects (font (size 1.27 1.27))))
 		(property "Manufacturer" "Murata" (at 274.32 181.61 0) (hide yes) (effects (font (size 1.27 1.27))))
+		(property "LCSC" "C86020" (at 274.32 181.61 0) (hide yes) (effects (font (size 1.27 1.27))))
 		(pin "1")
 		(pin "2")
@@
 		(property "MPN" "GRM188R71H104KA93D" (at 287.02 181.61 0) (hide yes) (effects (font (size 1.27 1.27))))
 		(property "Manufacturer" "Murata" (at 287.02 181.61 0) (hide yes) (effects (font (size 1.27 1.27))))
-		(pin "1")
-		(pin "2")
+		(property "LCSC" "C77055" (at 287.02 181.61 0) (hide yes) (effects (font (size 1.27 1.27))))
+		(pin "1")
+		(pin "2")

Commit message: Stage 3: footprints from datasheets and vendor libraries, 3D-checked (refs #3)
- ECE533_Mods.pretty (drawn from manufacturer datasheets):
  EPC2304 (EPC copper, solder-mask-defined land pattern and stencil),
  TDK ERUC23 (TDK recommended layout), R_2512_Kelvin (Bourns CSS2H-2512
  pads with net-tie sense strips), Littelfuse 456 fuse (+ placeholder STEP)
- ECE533_Vendor library (git-ignored): Wurth REDCUBE 74650194R and the
  SamacSys NME1S0505SC footprint; vendor STEP models referenced from
  kicad/lib/vendor, alignment verified by rendering
- gen_footprints.py regenerates both libraries; check_footprints.py checks
  symbol pins against footprint pads
- Fix D15/D16 BAT54W footprint: SOT-323, not SOD-323 (pin 3 had no pad)
- ERC: 0 violations locally (footprint links now resolve)

Co-Authored-By: Claude Opus 5.5 <noreply@anthropic.com>
Parts:
- PS1: footprint ECE533_Mods:Murata_NME1S_SIP-4 -> ECE533_Vendor:Murata_NME1S_SIP-4
Changed lines of the file:
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@@
 		(property "Reference" "PS1" (at 195.58 52.07 0) (effects (font (size 1.27 1.27)) (justify left)))
 		(property "Value" "NME1S0505SC" (at 195.58 60.96 0) (effects (font (size 1.27 1.27)) (justify left)))
-		(property "Footprint" "ECE533_Mods:Murata_NME1S_SIP-4" (at 203.2 55.88 0) (hide yes) (effects (font (size 1.27 1.27))))
+		(property "Footprint" "ECE533_Vendor:Murata_NME1S_SIP-4" (at 203.2 55.88 0) (hide yes) (effects (font (size 1.27 1.27))))
 		(property "Datasheet" "https://www.murata.com/products/productdata/8822286319646/KDC-NME1.pdf" (at 203.2 55.88 0) (hide yes) (effects (font (size 1.27 1.27))))
 		(property "Description" "1 W isolated DC/DC module, 5 V in, 5 V out, 1 kVDC" (at 203.2 55.88 0) (hide yes) (effects (font (size 1.27 1.27))))

Commit message: Stage 3: board set-up, JLCPCB rules and first-pass placement (refs #3)
- build_pcb.py builds the PCB from the netlist: ID-1 outline, 4 x 2 oz
  stack-up (3313, ENIG), layer names, LV_ISO/HV_SW net classes, heatsink,
  pedestal and fan-duct outlines, isolation-barrier rule area, and places
  all 273 footprints (power stage on the bottom under L1, isolators on the
  barrier column, terminals on the right edge)
- ECE533_Guide.kicad_dru: JLC 2 oz limits, HV margin, 2.5 mm barrier rule
- Test points 1.0 mm (all on top); L1 pin-1 mark moved off RS2
- DRC with parity: 0 errors; only unrouted nets and 1 silk warning remain
- docs/design/placement_stage3.md with renders, PROGRESS updated

Co-Authored-By: Claude Opus 5.5 <noreply@anthropic.com>
Parts:
- TP15, TP16: footprint TestPoint:TestPoint_Pad_D1.5mm -> TestPoint:TestPoint_Pad_D1.0mm
Changed lines of the file:
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@@
 		(property "Reference" "TP15" (at 266.7 49.53 0) (effects (font (size 1.27 1.27)) (justify left)))
 		(property "Value" "+5V_ISO" (at 266.7 52.07 0) (effects (font (size 1.27 1.27)) (justify left)))
-		(property "Footprint" "TestPoint:TestPoint_Pad_D1.5mm" (at 264.16 50.8 0) (hide yes) (effects (font (size 1.27 1.27))))
+		(property "Footprint" "TestPoint:TestPoint_Pad_D1.0mm" (at 264.16 50.8 0) (hide yes) (effects (font (size 1.27 1.27))))
 		(property "Datasheet" "" (at 264.16 50.8 0) (hide yes) (effects (font (size 1.27 1.27))))
 		(property "Description" "test point" (at 264.16 50.8 0) (hide yes) (effects (font (size 1.27 1.27))))
@@
 		(property "Reference" "TP16" (at 276.86 49.53 0) (effects (font (size 1.27 1.27)) (justify left)))
 		(property "Value" "GND_ISO" (at 276.86 52.07 0) (effects (font (size 1.27 1.27)) (justify left)))
-		(property "Footprint" "TestPoint:TestPoint_Pad_D1.5mm" (at 274.32 50.8 0) (hide yes) (effects (font (size 1.27 1.27))))
+		(property "Footprint" "TestPoint:TestPoint_Pad_D1.0mm" (at 274.32 50.8 0) (hide yes) (effects (font (size 1.27 1.27))))
 		(property "Datasheet" "" (at 274.32 50.8 0) (hide yes) (effects (font (size 1.27 1.27))))
 		(property "Description" "test point" (at 274.32 50.8 0) (hide yes) (effects (font (size 1.27 1.27))))
