File: kicad/ECE533_Guide/power_phase.kicad_sch (KiCad schematic)
At the start: 51 parts, among them Q3 EPC2304, Q4 EPC2304, U1 Si8274GB1-IS1, U6 AMC3301, U9 INA301A3

Commit message: Stage 2: BOM from schematic, LCSC numbers, fix duplicate C114 (refs #2)
- kicad/tools/make_bom.py builds bom/PCB_BOM.xlsx (+ CSV) from the netlist;
  previous report BOM kept as a sheet, Digi-Key PNs carried over
- 47 LCSC numbers verified on lcsc.com; two unconfirmed Murata MPNs replaced
- check_netlist.py now also checks for duplicate reference designators
- Yageo part-number codes fixed (13K, 0R jumper)

Co-Authored-By: Claude Opus 5.5 <noreply@anthropic.com>
Parts:
- C11, C30, C40, C45, C47, C49, C50, C7, C8: LCSC (none) -> C77055
- C12: LCSC (none) -> C86038
- C32, C33: LCSC (none) -> C162275
- C36, C37: LCSC (none) -> C2170811; MPN GRM21A5C2D102JW01D -> C0805C102J2GAC7800; Manufacturer Murata -> KEMET
- C42: LCSC (none) -> C77026
- C43, C44, C46, C48: LCSC (none) -> C86020
Changed lines of the file:
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@@
 		(property "MPN" "GRM188R71H104KA93D" (at 91.44 87.63 0) (hide yes) (effects (font (size 1.27 1.27))))
 		(property "Manufacturer" "Murata" (at 91.44 87.63 0) (hide yes) (effects (font (size 1.27 1.27))))
+		(property "LCSC" "C77055" (at 91.44 87.63 0) (hide yes) (effects (font (size 1.27 1.27))))
 		(pin "1")
 		(pin "2")
@@
 		(property "MPN" "GRM188R71H104KA93D" (at 60.96 107.95 0) (hide yes) (effects (font (size 1.27 1.27))))
 		(property "Manufacturer" "Murata" (at 60.96 107.95 0) (hide yes) (effects (font (size 1.27 1.27))))
+		(property "LCSC" "C77055" (at 60.96 107.95 0) (hide yes) (effects (font (size 1.27 1.27))))
 		(pin "1")
 		(pin "2")
@@
 		(property "MPN" "GRM188R71H104KA93D" (at 172.72 59.69 0) (hide yes) (effects (font (size 1.27 1.27))))
 		(property "Manufacturer" "Murata" (at 172.72 59.69 0) (hide yes) (effects (font (size 1.27 1.27))))
+		(property "LCSC" "C77055" (at 172.72 59.69 0) (hide yes) (effects (font (size 1.27 1.27))))
 		(pin "1")
 		(pin "2")
@@
 		(property "MPN" "GRM188R71H104KA93D" (at 177.8 105.41 0) (hide yes) (effects (font (size 1.27 1.27))))
 		(property "Manufacturer" "Murata" (at 177.8 105.41 0) (hide yes) (effects (font (size 1.27 1.27))))
+		(property "LCSC" "C77055" (at 177.8 105.41 0) (hide yes) (effects (font (size 1.27 1.27))))
 		(pin "1")
 		(pin "2")
@@
 		(property "MPN" "GRM21BR71A106KE51L" (at 190.5 105.41 0) (hide yes) (effects (font (size 1.27 1.27))))
 		(property "Manufacturer" "Murata" (at 190.5 105.41 0) (hide yes) (effects (font (size 1.27 1.27))))
+		(property "LCSC" "C86038" (at 190.5 105.41 0) (hide yes) (effects (font (size 1.27 1.27))))
 		(pin "1")
 		(pin "2")
@@
 		(property "Datasheet" "" (at 294.64 67.31 0) (hide yes) (effects (font (size 1.27 1.27))))
 		(property "Description" "Unpolarized capacitor" (at 294.64 67.31 0) (hide yes) (effects (font (size 1.27 1.27))))
-		(property "MPN" "GRM21A5C2D102JW01D" (at 294.64 67.31 0) (hide yes) (effects (font (size 1.27 1.27))))
-		(property "Manufacturer" "Murata" (at 294.64 67.31 0) (hide yes) (effects (font (size 1.27 1.27))))
+		(property "MPN" "C0805C102J2GAC7800" (at 294.64 67.31 0) (hide yes) (effects (font (size 1.27 1.27))))
+		(property "Manufacturer" "KEMET" (at 294.64 67.31 0) (hide yes) (effects (font (size 1.27 1.27))))
+		(property "LCSC" "C2170811" (at 294.64 67.31 0) (hide yes) (effects (font (size 1.27 1.27))))
 		(pin "1")
 		(pin "2")
@@
 		(property "Datasheet" "" (at 294.64 123.19 0) (hide yes) (effects (font (size 1.27 1.27))))
 		(property "Description" "Unpolarized capacitor" (at 294.64 123.19 0) (hide yes) (effects (font (size 1.27 1.27))))
-		(property "MPN" "GRM21A5C2D102JW01D" (at 294.64 123.19 0) (hide yes) (effects (font (size 1.27 1.27))))
-		(property "Manufacturer" "Murata" (at 294.64 123.19 0) (hide yes) (effects (font (size 1.27 1.27))))
+		(property "MPN" "C0805C102J2GAC7800" (at 294.64 123.19 0) (hide yes) (effects (font (size 1.27 1.27))))
+		(property "Manufacturer" "KEMET" (at 294.64 123.19 0) (hide yes) (effects (font (size 1.27 1.27))))
+		(property "LCSC" "C2170811" (at 294.64 123.19 0) (hide yes) (effects (font (size 1.27 1.27))))
 		(pin "1")
 		(pin "2")
@@
 		(property "MPN" "GRM188R72A103KA01D" (at 340.36 95.25 0) (hide yes) (effects (font (size 1.27 1.27))))
 		(property "Manufacturer" "Murata" (at 340.36 95.25 0) (hide yes) (effects (font (size 1.27 1.27))))
+		(property "LCSC" "C162275" (at 340.36 95.25 0) (hide yes) (effects (font (size 1.27 1.27))))
 		(pin "1")
 		(pin "2")
@@
 		(property "MPN" "GRM188R72A103KA01D" (at 355.6 95.25 0) (hide yes) (effects (font (size 1.27 1.27))))
 		(property "Manufacturer" "Murata" (at 355.6 95.25 0) (hide yes) (effects (font (size 1.27 1.27))))
+		(property "LCSC" "C162275" (at 355.6 95.25 0) (hide yes) (effects (font (size 1.27 1.27))))
 		(pin "1")
 		(pin "2")
@@
 		(property "MPN" "GRM188R71H104KA93D" (at 340.36 181.61 0) (hide yes) (effects (font (size 1.27 1.27))))
 		(property "Manufacturer" "Murata" (at 340.36 181.61 0) (hide yes) (effects (font (size 1.27 1.27))))
+		(property "LCSC" "C77055" (at 340.36 181.61 0) (hide yes) (effects (font (size 1.27 1.27))))
 		(pin "1")
 		(pin "2")
@@
 		(property "MPN" "GRM1885C1H102JA01D" (at 223.52 227.33 0) (hide yes) (effects (font (size 1.27 1.27))))
 		(property "Manufacturer" "Murata" (at 223.52 227.33 0) (hide yes) (effects (font (size 1.27 1.27))))
+		(property "LCSC" "C77026" (at 223.52 227.33 0) (hide yes) (effects (font (size 1.27 1.27))))
 		(pin "1")
 		(pin "2")
@@
 		(property "MPN" "GRM188R71E105KA12D" (at 167.64 176.53 0) (hide yes) (effects (font (size 1.27 1.27))))
 		(property "Manufacturer" "Murata" (at 167.64 176.53 0) (hide yes) (effects (font (size 1.27 1.27))))
+		(property "LCSC" "C86020" (at 167.64 176.53 0) (hide yes) (effects (font (size 1.27 1.27))))
 		(pin "1")
 		(pin "2")
@@
 		(property "MPN" "GRM188R71H104KA93D" (at 180.34 176.53 0) (hide yes) (effects (font (size 1.27 1.27))))
 		(property "Manufacturer" "Murata" (at 180.34 176.53 0) (hide yes) (effects (font (size 1.27 1.27))))
+		(property "LCSC" "C77055" (at 180.34 176.53 0) (hide yes) (effects (font (size 1.27 1.27))))
 		(pin "1")
 		(pin "2")
@@
 		(property "MPN" "GRM188R71E105KA12D" (at 193.04 176.53 0) (hide yes) (effects (font (size 1.27 1.27))))
 		(property "Manufacturer" "Murata" (at 193.04 176.53 0) (hide yes) (effects (font (size 1.27 1.27))))
+		(property "LCSC" "C86020" (at 193.04 176.53 0) (hide yes) (effects (font (size 1.27 1.27))))
 		(pin "1")
 		(pin "2")
@@
 		(property "MPN" "GRM188R71H104KA93D" (at 205.74 176.53 0) (hide yes) (effects (font (size 1.27 1.27))))
 		(property "Manufacturer" "Murata" (at 205.74 176.53 0) (hide yes) (effects (font (size 1.27 1.27))))
+		(property "LCSC" "C77055" (at 205.74 176.53 0) (hide yes) (effects (font (size 1.27 1.27))))
 		(pin "1")
 		(pin "2")
@@
 		(property "MPN" "GRM188R71E105KA12D" (at 50.8 176.53 0) (hide yes) (effects (font (size 1.27 1.27))))
 		(property "Manufacturer" "Murata" (at 50.8 176.53 0) (hide yes) (effects (font (size 1.27 1.27))))
+		(property "LCSC" "C86020" (at 50.8 176.53 0) (hide yes) (effects (font (size 1.27 1.27))))
 		(pin "1")
 		(pin "2")
@@
 		(property "MPN" "GRM188R71H104KA93D" (at 63.5 176.53 0) (hide yes) (effects (font (size 1.27 1.27))))
 		(property "Manufacturer" "Murata" (at 63.5 176.53 0) (hide yes) (effects (font (size 1.27 1.27))))
+		(property "LCSC" "C77055" (at 63.5 176.53 0) (hide yes) (effects (font (size 1.27 1.27))))
 		(pin "1")
 		(pin "2")
@@
 		(property "MPN" "GRM188R71E105KA12D" (at 76.2 176.53 0) (hide yes) (effects (font (size 1.27 1.27))))
 		(property "Manufacturer" "Murata" (at 76.2 176.53 0) (hide yes) (effects (font (size 1.27 1.27))))
+		(property "LCSC" "C86020" (at 76.2 176.53 0) (hide yes) (effects (font (size 1.27 1.27))))
 		(pin "1")
 		(pin "2")
@@
 		(property "MPN" "GRM188R71H104KA93D" (at 88.9 176.53 0) (hide yes) (effects (font (size 1.27 1.27))))
 		(property "Manufacturer" "Murata" (at 88.9 176.53 0) (hide yes) (effects (font (size 1.27 1.27))))
-		(pin "1")
-		(pin "2")
+		(property "LCSC" "C77055" (at 88.9 176.53 0) (hide yes) (effects (font (size 1.27 1.27))))
+		(pin "1")
+		(pin "2")

Commit message: Stage 3: board set-up, JLCPCB rules and first-pass placement (refs #3)
- build_pcb.py builds the PCB from the netlist: ID-1 outline, 4 x 2 oz
  stack-up (3313, ENIG), layer names, LV_ISO/HV_SW net classes, heatsink,
  pedestal and fan-duct outlines, isolation-barrier rule area, and places
  all 273 footprints (power stage on the bottom under L1, isolators on the
  barrier column, terminals on the right edge)
- ECE533_Guide.kicad_dru: JLC 2 oz limits, HV margin, 2.5 mm barrier rule
- Test points 1.0 mm (all on top); L1 pin-1 mark moved off RS2
- DRC with parity: 0 errors; only unrouted nets and 1 silk warning remain
- docs/design/placement_stage3.md with renders, PROGRESS updated

Co-Authored-By: Claude Opus 5.5 <noreply@anthropic.com>
Parts:
- TP3, TP5, TP6, TP9: footprint TestPoint:TestPoint_Pad_D1.5mm -> TestPoint:TestPoint_Pad_D1.0mm
Changed lines of the file:
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@@
 		(property "Reference" "TP3" (at 266.7 90.17 0) (effects (font (size 1.27 1.27)) (justify left)))
 		(property "Value" "SW" (at 266.7 92.71 0) (effects (font (size 1.27 1.27)) (justify left)))
-		(property "Footprint" "TestPoint:TestPoint_Pad_D1.5mm" (at 264.16 91.44 0) (hide yes) (effects (font (size 1.27 1.27))))
+		(property "Footprint" "TestPoint:TestPoint_Pad_D1.0mm" (at 264.16 91.44 0) (hide yes) (effects (font (size 1.27 1.27))))
 		(property "Datasheet" "" (at 264.16 91.44 0) (hide yes) (effects (font (size 1.27 1.27))))
 		(property "Description" "test point" (at 264.16 91.44 0) (hide yes) (effects (font (size 1.27 1.27))))
@@
 		(property "Reference" "TP5" (at 243.84 69.85 0) (effects (font (size 1.27 1.27)) (justify left)))
 		(property "Value" "GH gate" (at 243.84 72.39 0) (effects (font (size 1.27 1.27)) (justify left)))
-		(property "Footprint" "TestPoint:TestPoint_Pad_D1.5mm" (at 241.3 71.12 0) (hide yes) (effects (font (size 1.27 1.27))))
+		(property "Footprint" "TestPoint:TestPoint_Pad_D1.0mm" (at 241.3 71.12 0) (hide yes) (effects (font (size 1.27 1.27))))
 		(property "Datasheet" "" (at 241.3 71.12 0) (hide yes) (effects (font (size 1.27 1.27))))
 		(property "Description" "test point" (at 241.3 71.12 0) (hide yes) (effects (font (size 1.27 1.27))))
@@
 		(property "Reference" "TP6" (at 243.84 125.73 0) (effects (font (size 1.27 1.27)) (justify left)))
 		(property "Value" "GL gate" (at 243.84 128.27 0) (effects (font (size 1.27 1.27)) (justify left)))
-		(property "Footprint" "TestPoint:TestPoint_Pad_D1.5mm" (at 241.3 127 0) (hide yes) (effects (font (size 1.27 1.27))))
+		(property "Footprint" "TestPoint:TestPoint_Pad_D1.0mm" (at 241.3 127 0) (hide yes) (effects (font (size 1.27 1.27))))
 		(property "Datasheet" "" (at 241.3 127 0) (hide yes) (effects (font (size 1.27 1.27))))
 		(property "Description" "test point" (at 241.3 127 0) (hide yes) (effects (font (size 1.27 1.27))))
@@
 		(property "Reference" "TP9" (at 378.46 186.69 0) (effects (font (size 1.27 1.27)) (justify left)))
 		(property "Value" "IMON" (at 378.46 189.23 0) (effects (font (size 1.27 1.27)) (justify left)))
-		(property "Footprint" "TestPoint:TestPoint_Pad_D1.5mm" (at 375.92 187.96 0) (hide yes) (effects (font (size 1.27 1.27))))
+		(property "Footprint" "TestPoint:TestPoint_Pad_D1.0mm" (at 375.92 187.96 0) (hide yes) (effects (font (size 1.27 1.27))))
 		(property "Datasheet" "" (at 375.92 187.96 0) (hide yes) (effects (font (size 1.27 1.27))))
 		(property "Description" "test point" (at 375.92 187.96 0) (hide yes) (effects (font (size 1.27 1.27))))
