File: kicad/ECE533_Guide/power_stage.kicad_sch (KiCad schematic)
At the start: 23 parts, among them J2 VOUT+, J6 VOUT-, U14 TLV3012

Commit message: Stage 2: BOM from schematic, LCSC numbers, fix duplicate C114 (refs #2)
- kicad/tools/make_bom.py builds bom/PCB_BOM.xlsx (+ CSV) from the netlist;
  previous report BOM kept as a sheet, Digi-Key PNs carried over
- 47 LCSC numbers verified on lcsc.com; two unconfirmed Murata MPNs replaced
- check_netlist.py now also checks for duplicate reference designators
- Yageo part-number codes fixed (13K, 0R jumper)

Co-Authored-By: Claude Opus 5.5 <noreply@anthropic.com>
Parts:
- C60, C61, C62, C63, C64, C65: LCSC (none) -> C77102
- C68: LCSC (none) -> C77055
- FB1: LCSC (none) -> C85833
- R42: MPN RC0603FR-070RL -> RC0603JR-070RL
Changed lines of the file:
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@@
 		(property "MPN" "GRM32ER71H106KA12L" (at 243.84 59.69 0) (hide yes) (effects (font (size 1.27 1.27))))
 		(property "Manufacturer" "Murata" (at 243.84 59.69 0) (hide yes) (effects (font (size 1.27 1.27))))
+		(property "LCSC" "C77102" (at 243.84 59.69 0) (hide yes) (effects (font (size 1.27 1.27))))
 		(pin "1")
 		(pin "2")
@@
 		(property "MPN" "GRM32ER71H106KA12L" (at 254 59.69 0) (hide yes) (effects (font (size 1.27 1.27))))
 		(property "Manufacturer" "Murata" (at 254 59.69 0) (hide yes) (effects (font (size 1.27 1.27))))
+		(property "LCSC" "C77102" (at 254 59.69 0) (hide yes) (effects (font (size 1.27 1.27))))
 		(pin "1")
 		(pin "2")
@@
 		(property "MPN" "GRM32ER71H106KA12L" (at 264.16 59.69 0) (hide yes) (effects (font (size 1.27 1.27))))
 		(property "Manufacturer" "Murata" (at 264.16 59.69 0) (hide yes) (effects (font (size 1.27 1.27))))
+		(property "LCSC" "C77102" (at 264.16 59.69 0) (hide yes) (effects (font (size 1.27 1.27))))
 		(pin "1")
 		(pin "2")
@@
 		(property "MPN" "GRM32ER71H106KA12L" (at 274.32 59.69 0) (hide yes) (effects (font (size 1.27 1.27))))
 		(property "Manufacturer" "Murata" (at 274.32 59.69 0) (hide yes) (effects (font (size 1.27 1.27))))
+		(property "LCSC" "C77102" (at 274.32 59.69 0) (hide yes) (effects (font (size 1.27 1.27))))
 		(pin "1")
 		(pin "2")
@@
 		(property "MPN" "GRM32ER71H106KA12L" (at 284.48 59.69 0) (hide yes) (effects (font (size 1.27 1.27))))
 		(property "Manufacturer" "Murata" (at 284.48 59.69 0) (hide yes) (effects (font (size 1.27 1.27))))
+		(property "LCSC" "C77102" (at 284.48 59.69 0) (hide yes) (effects (font (size 1.27 1.27))))
 		(pin "1")
 		(pin "2")
@@
 		(property "MPN" "GRM32ER71H106KA12L" (at 294.64 59.69 0) (hide yes) (effects (font (size 1.27 1.27))))
 		(property "Manufacturer" "Murata" (at 294.64 59.69 0) (hide yes) (effects (font (size 1.27 1.27))))
+		(property "LCSC" "C77102" (at 294.64 59.69 0) (hide yes) (effects (font (size 1.27 1.27))))
 		(pin "1")
 		(pin "2")
@@
 		(property "MPN" "GRM188R71H104KA93D" (at 330.2 135.89 0) (hide yes) (effects (font (size 1.27 1.27))))
 		(property "Manufacturer" "Murata" (at 330.2 135.89 0) (hide yes) (effects (font (size 1.27 1.27))))
+		(property "LCSC" "C77055" (at 330.2 135.89 0) (hide yes) (effects (font (size 1.27 1.27))))
 		(pin "1")
 		(pin "2")
@@
 		(property "MPN" "BLM18KG601SN1D" (at 162.56 147.32 0) (hide yes) (effects (font (size 1.27 1.27))))
 		(property "Manufacturer" "Murata" (at 162.56 147.32 0) (hide yes) (effects (font (size 1.27 1.27))))
+		(property "LCSC" "C85833" (at 162.56 147.32 0) (hide yes) (effects (font (size 1.27 1.27))))
 		(pin "1")
 		(pin "2")
@@
 		(property "Datasheet" "" (at 177.8 156.21 0) (hide yes) (effects (font (size 1.27 1.27))))
 		(property "Description" "Resistor" (at 177.8 156.21 0) (hide yes) (effects (font (size 1.27 1.27))))
-		(property "MPN" "RC0603FR-070RL" (at 177.8 156.21 0) (hide yes) (effects (font (size 1.27 1.27))))
+		(property "MPN" "RC0603JR-070RL" (at 177.8 156.21 0) (hide yes) (effects (font (size 1.27 1.27))))
 		(property "Manufacturer" "YAGEO" (at 177.8 156.21 0) (hide yes) (effects (font (size 1.27 1.27))))
 		(pin "1")

Commit message: Stage 3: footprints from datasheets and vendor libraries, 3D-checked (refs #3)
- ECE533_Mods.pretty (drawn from manufacturer datasheets):
  EPC2304 (EPC copper, solder-mask-defined land pattern and stencil),
  TDK ERUC23 (TDK recommended layout), R_2512_Kelvin (Bourns CSS2H-2512
  pads with net-tie sense strips), Littelfuse 456 fuse (+ placeholder STEP)
- ECE533_Vendor library (git-ignored): Wurth REDCUBE 74650194R and the
  SamacSys NME1S0505SC footprint; vendor STEP models referenced from
  kicad/lib/vendor, alignment verified by rendering
- gen_footprints.py regenerates both libraries; check_footprints.py checks
  symbol pins against footprint pads
- Fix D15/D16 BAT54W footprint: SOT-323, not SOD-323 (pin 3 had no pad)
- ERC: 0 violations locally (footprint links now resolve)

Co-Authored-By: Claude Opus 5.5 <noreply@anthropic.com>
Parts:
- J2, J6: footprint ECE533_Mods:Wurth_REDCUBE_74650194 -> ECE533_Vendor:Wurth_REDCUBE_74650194
Changed lines of the file:
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@@
 		(property "Reference" "J2" (at 368.3 54.61 0) (effects (font (size 1.27 1.27)) (justify left)))
 		(property "Value" "VOUT+" (at 368.3 57.15 0) (effects (font (size 1.27 1.27)) (justify left)))
-		(property "Footprint" "ECE533_Mods:Wurth_REDCUBE_74650194" (at 365.76 55.88 0) (hide yes) (effects (font (size 1.27 1.27))))
+		(property "Footprint" "ECE533_Vendor:Wurth_REDCUBE_74650194" (at 365.76 55.88 0) (hide yes) (effects (font (size 1.27 1.27))))
 		(property "Datasheet" "" (at 365.76 55.88 0) (hide yes) (effects (font (size 1.27 1.27))))
 		(property "Description" "Generic connector, single row, 01x01, script generated (kicad-library-utils/schlib/autogen/connector/)" (at 365.76 55.88 0) (hide yes) (effects (font (size 1.27 1.27))))
@@
 		(property "Reference" "J6" (at 368.3 69.85 0) (effects (font (size 1.27 1.27)) (justify left)))
 		(property "Value" "VOUT-" (at 368.3 72.39 0) (effects (font (size 1.27 1.27)) (justify left)))
-		(property "Footprint" "ECE533_Mods:Wurth_REDCUBE_74650194" (at 365.76 71.12 0) (hide yes) (effects (font (size 1.27 1.27))))
+		(property "Footprint" "ECE533_Vendor:Wurth_REDCUBE_74650194" (at 365.76 71.12 0) (hide yes) (effects (font (size 1.27 1.27))))
 		(property "Datasheet" "" (at 365.76 71.12 0) (hide yes) (effects (font (size 1.27 1.27))))
 		(property "Description" "Generic connector, single row, 01x01, script generated (kicad-library-utils/schlib/autogen/connector/)" (at 365.76 71.12 0) (hide yes) (effects (font (size 1.27 1.27))))

Commit message: Stage 3: board set-up, JLCPCB rules and first-pass placement (refs #3)
- build_pcb.py builds the PCB from the netlist: ID-1 outline, 4 x 2 oz
  stack-up (3313, ENIG), layer names, LV_ISO/HV_SW net classes, heatsink,
  pedestal and fan-duct outlines, isolation-barrier rule area, and places
  all 273 footprints (power stage on the bottom under L1, isolators on the
  barrier column, terminals on the right edge)
- ECE533_Guide.kicad_dru: JLC 2 oz limits, HV margin, 2.5 mm barrier rule
- Test points 1.0 mm (all on top); L1 pin-1 mark moved off RS2
- DRC with parity: 0 errors; only unrouted nets and 1 silk warning remain
- docs/design/placement_stage3.md with renders, PROGRESS updated

Co-Authored-By: Claude Opus 5.5 <noreply@anthropic.com>
Parts:
- TP2: footprint TestPoint:TestPoint_Pad_D1.5mm -> TestPoint:TestPoint_Pad_D1.0mm
Changed lines of the file:
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@@
 		(property "Reference" "TP2" (at 261.62 95.25 0) (effects (font (size 1.27 1.27)) (justify left)))
 		(property "Value" "VOUT" (at 261.62 97.79 0) (effects (font (size 1.27 1.27)) (justify left)))
-		(property "Footprint" "TestPoint:TestPoint_Pad_D1.5mm" (at 259.08 96.52 0) (hide yes) (effects (font (size 1.27 1.27))))
+		(property "Footprint" "TestPoint:TestPoint_Pad_D1.0mm" (at 259.08 96.52 0) (hide yes) (effects (font (size 1.27 1.27))))
 		(property "Datasheet" "" (at 259.08 96.52 0) (hide yes) (effects (font (size 1.27 1.27))))
 		(property "Description" "test point" (at 259.08 96.52 0) (hide yes) (effects (font (size 1.27 1.27))))
