File: kicad/PowerModule/PowerModule.kicad_sch (KiCad schematic)
At the start: 14 parts, among them J1 DC+, J2 Power_out, J3 DC-, Q3 EPC2304, Q4 EPC2304, Q5 EPC2304, Q6 EPC2304

Commit message: Power module: bulk caps split into 4 x 62 uF, J4 centred with fixed control lanes
- C5/C6 -> C5+C15 (output), C6+C16 (input): 2 x EGXF161ELL620MJ25S per position (user: half
  values for lower ESR); VIN/VOUT labels added (pm_split_bulk.py), ERC 0 errors
- J4 centred on the left edge; AT1 pair on L4, AT2 pair on L1, +5V lane on L4: 15-19 mm per
  command line, no meanders; PS1 to the bottom left, H2 screw to (28.4, 50.6)
- PS1 barrier keep-out from pin-2 to pin-3 centre (1.5 mm per side)
- name block on the bottom silkscreen auto-sized into the clear strip (2.0 mm)
- DRC with schematic parity: 0 violations, 0 unconnected, 0 parity issues

Co-Authored-By: Claude Opus 5.5 <noreply@anthropic.com>
Parts:
- added C15: 62u/160V, Capacitor_THT:CP_Radial_D10.0mm_P5.00mm, symbol Device:C_Small
- added C16: 62u/160V, Capacitor_THT:CP_Radial_D10.0mm_P5.00mm, symbol Device:C_Small_US
- C5, C6: value 110u/160V -> 62u/160V; footprint Capacitor_THT:CP_Radial_D12.5mm_P5.00mm -> Capacitor_THT:CP_Radial_D10.0mm_P5.00mm; LCSC C1598290 -> (none); MPN EGXF161ELL111MK25S -> EGXF161ELL620MJ25S
Connections:
- net GNDPWR: now also C15.2, C16.2
- net VIN: now reaches C1.1, C3.1, C6.1, J1.1 (Pin_1), Q3.10 (D_6), Q3.11 (D_7), Q3.3 (D_1), Q3.5 (D_2), Q3.7 (D_3), Q3.8 (D_4), Q3.9 (D_5), Q6.10 (D_6), Q6.11 (D_7), Q6.3 (D_1), Q6.5 (D_2), Q6.7 (D_3), Q6.8 (D_4), Q6.9 (D_5)
- net VIN: now also C16.1
- net VOUT: now reaches C5.1, J2.1 (Pin_1), L1.1, L1.2
- net VOUT: now also C15.1
