File: kicad/PowerModule/gate_drive.kicad_sch (KiCad schematic)
At the start: 40 parts, among them J4 105313-1206, U1 1EDN7550B, U2 1EDN7550B, U3 1EDN7550B, U4 1EDN7550B

Commit message: Power module: symmetric bulk caps, PS1 centred on J4, right-angle J4 with model
- bulk caps mirror-symmetric: C6/C16 on the top edge (VBUS), C5/C15 on the bottom edge (VOUT
  strip added), x 37.5 / 64.6; PGND tongues for C6 (L1 + vias) and C16
- PS1 on J4's centreline; J4 right angle, mating face 2.2 mm off the edge; H2 back to (21.5, 50)
- J4 project footprint Molex_Nano-Fit_105313-1206_RA (off-board silk dropped) + generated
  right-angle STEP (gen_footprints.py, nanofit_fp.py)
- name block 2.35 mm in the widened clear strip
- ERC 0 errors; DRC with schematic parity: 0 violations, 0 unconnected, 0 parity issues

Co-Authored-By: Claude Opus 5.5 <noreply@anthropic.com>
Parts:
- J4: footprint Connector_Molex:Molex_Nano-Fit_105313-xx06_1x06_P2.50mm_Horizontal -> ECE533_Mods:Molex_Nano-Fit_105313-1206_RA
Changed lines of the file:
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@@
 			)
 		)
-		(property "Footprint" "Connector_Molex:Molex_Nano-Fit_105313-xx06_1x06_P2.50mm_Horizontal"
+		(property "Footprint" "ECE533_Mods:Molex_Nano-Fit_105313-1206_RA"
 			(at 15.24 16.84 0)
 			(hide yes)

Commit message: Power module: 1 kOhm gate pull-downs R21-R24 at the gate pads
- schematic: R21 P1H-KS1, R22 P1L-GNDPWR, R23 P2H-KS2, R24 P2L-GNDPWR (pm_pulldowns.py), as in
  the report's LTspice model; ERC 0 errors
- HS pull-downs on the bottom inside the Kelvin island next to the gate pads, LS on the top over
  the gate via next to the LS Kelvin via
- DRC with schematic parity: 0 violations, 0 unconnected, 0 parity issues; BOM and docs updated

Co-Authored-By: Claude Opus 5.5 <noreply@anthropic.com>
Parts:
- added R21, R22, R23, R24: 1k, Resistor_SMD:R_0603_1608Metric, symbol Device:R_Small_US
Connections:
- net GNDPWR: now also R22.2, R24.2
- net KS1: now also R21.2
- net KS2: now also R23.2
- net P1H: now also R21.1
- net P1L: now also R22.1
- net P2H: now also R23.1
- net P2L: now also R24.1
